Commit message: add arm to cob_body

File: urdf/cob4-25_0412_torso.urdf (robot description, URDF)
Before this commit: robot tricycle_drive, 19 links, 18 joints
Joints:
- joint torso_base_joint: origin xyz=0.0 0.0 0.26411 rpy=0.0 0.0 0.0 -> xyz=0.0 0.0 0.26411 rpy=0.0 0.0 3.1416

File: urdf/cob4-25_0412_torso_cam.urdf (robot description, URDF)
Before this commit: robot tricycle_drive, 33 links, 32 joints
Joints:
- joint torso_base_joint: origin xyz=0.0 0.0 0.26411 rpy=0.0 0.0 0.0 -> xyz=0.0 0.0 0.26411 rpy=0.0 0.0 3.1416
